File: baseplate.kicad_pcb (KiCad board)
At the start: 2 copper layers, 243.8 x 114.3 mm, 7 parts

Commit message: edit baseplate
Parts:
- removed the REF** at (48.3, 83.8)
- removed the REF** at (251.5, 124.5)
- removed the REF** at (48.3, 124.5)
- removed the REF** at (251.5, 83.8)
- added REF**: M2_Hole_TH, kbd:M2_Hole_TH, F.Cu at (47.6, 123.1)
- added REF**: M2_Hole_TH, kbd:M2_Hole_TH, F.Cu at (238.1, 123.1)
- added REF**: M2_Hole_TH, kbd:M2_Hole_TH, F.Cu at (238.1, 85.0)
- added REF**: M2_Hole_TH, kbd:M2_Hole_TH, F.Cu at (47.6, 85.0)
- moved REF** 14.0 mm to (254.3, 34.0)
- moved REF** 0.13 mm to (31.5, 34.0)
Other:
- board size 243.8 x 114.3 mm -> 229.9 x 112.2 mm
- board text added: "112.25mm"
- board text added: "229.852mm"
- board text removed: "114.30mm"
- board text removed: "243.84mm"
Changed lines of the file:
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@@
   (net 0 "")
   (footprint "kbd:M2_Hole_TH" (layer "F.Cu")
-    (at 31.496 33.909)
+    (at 47.625 123.063)
+    (attr through_hole)
+    (fp_text reference "REF**" (at 0 0.5) (layer "F.SilkS")
+      (effects (font (size 1 1) (thickness 0.15)))
+    )
+    (fp_text value "M2_Hole_TH" (at 0 -0.5) (layer "F.Fab")
+      (effects (font (size 1 1) (thickness 0.15)))
+    )
+    (pad "" thru_hole circle locked (at 0 0) (size 4.2 4.2) (drill 2.3) (layers *.Cu *.Mask))
+  )
+  (footprint "kbd:M2_Hole_TH" (layer "F.Cu")
+    (at 238.125 123.063)
+    (attr through_hole)
+    (fp_text reference "REF**" (at 0 0.5) (layer "F.SilkS")
+      (effects (font (size 1 1) (thickness 0.15)))
+    )
+    (fp_text value "M2_Hole_TH" (at 0 -0.5) (layer "F.Fab")
+      (effects (font (size 1 1) (thickness 0.15)))
+    )
+    (pad "" thru_hole circle locked (at 0 0) (size 4.2 4.2) (drill 2.3) (layers *.Cu *.Mask))
+  )
+  (footprint "kbd:M2_Hole_TH" (layer "F.Cu")
+    (at 31.496 34.036)
     (attr through_hole)
     (fp_text reference "REF**" (at 0 0.5) (layer "F.SilkS") hide
@@
   )
   (footprint "kbd:M2_Hole_TH" (layer "F.Cu")
-    (at 268.224 34.036)
+    (at 254.254 34.036)
     (attr through_hole)
     (fp_text reference "REF**" (at 0 0.5) (layer "F.SilkS") hide
@@
   )
   (footprint "kbd:M2_Hole_TH" (layer "F.Cu")
-    (at 48.26 83.82)
-    (attr through_hole)
-    (fp_text reference "REF**" (at 0 0.5) (layer "F.SilkS")
-      (effects (font (size 1 1) (thickness 0.15)))
-    )
-    (fp_text value "M2_Hole_TH" (at 0 -0.5) (layer "F.Fab")
-      (effects (font (size 1 1) (thickness 0.15)))
-    )
-    (pad "" thru_hole circle locked (at 0 0) (size 4.2 4.2) (drill 2.3) (layers *.Cu *.Mask))
-  )
-  (footprint "kbd:M2_Hole_TH" (layer "F.Cu")
-    (at 251.46 124.46)
+    (at 238.125 84.963)
     (attr through_hole)
     (fp_text reference "REF**" (at 0 0.5) (layer "F.SilkS")
@@
   )
   (footprint "kbd:M2_Hole_TH" (layer "F.Cu")
-    (at 48.26 124.46)
-    (attr through_hole)
-    (fp_text reference "REF**" (at 0 0.5) (layer "F.SilkS")
-      (effects (font (size 1 1) (thickness 0.15)))
-    )
-    (fp_text value "M2_Hole_TH" (at 0 -0.5) (layer "F.Fab")
-      (effects (font (size 1 1) (thickness 0.15)))
-    )
-    (pad "" thru_hole circle locked (at 0 0) (size 4.2 4.2) (drill 2.3) (layers *.Cu *.Mask))
-  )
-  (footprint "kbd:M2_Hole_TH" (layer "F.Cu")
-    (at 251.46 83.82)
+    (at 47.625 84.963)
     (attr through_hole)
     (fp_text reference "REF**" (at 0 0.5) (layer "F.SilkS")
@@
   )
   (gr_line (start 27.94 151.13) (end 27.94 156.21) (layer "Eco1.User") (width 0.5))
-  (gr_line (start 27.94 153.67) (end 271.78 153.67) (layer "Eco1.User") (width 0.5))
+  (gr_line (start 27.94 153.67) (end 257.81 153.67) (layer "Eco1.User") (width 0.5))
   (gr_line (start 276.86 30.48) (end 281.94 30.48) (layer "Eco1.User") (width 0.5))
-  (gr_line (start 279.4 30.48) (end 279.4 144.78) (layer "Eco1.User") (width 0.5))
-  (gr_line (start 276.86 144.78) (end 281.94 144.78) (layer "Eco1.User") (width 0.5))
-  (gr_line (start 271.78 151.13) (end 271.78 156.21) (layer "Eco1.User") (width 0.5))
-  (gr_arc (start 271.78 142.24) (mid 271.036051 144.036051) (end 269.24 144.78) (layer "Edge.Cuts") (width 0.1))
-  (gr_line (start 269.24 144.78) (end 30.48 144.78) (layer "Edge.Cuts") (width 0.05))
-  (gr_line (start 30.48 30.48) (end 269.24 30.48) (layer "Edge.Cuts") (width 0.1))
+  (gr_line (start 279.4 30.48) (end 279.4 142.748) (layer "Eco1.User") (width 0.5))
+  (gr_line (start 276.86 142.748) (end 281.94 142.748) (layer "Eco1.User") (width 0.5))
+  (gr_line (start 257.81 151.13) (end 257.81 156.21) (layer "Eco1.User") (width 0.5))
+  (gr_arc (start 257.791949 140.189949) (mid 257.048 141.986) (end 255.251949 142.729949) (layer "Edge.Cuts") (width 0.1))
+  (gr_line (start 255.251949 142.729949) (end 30.48 142.729949) (layer "Edge.Cuts") (width 0.1))
+  (gr_line (start 30.48 30.48) (end 255.251949 30.48) (layer "Edge.Cuts") (width 0.1))
   (gr_arc (start 27.94 33.02) (mid 28.683949 31.223949) (end 30.48 30.48) (layer "Edge.Cuts") (width 0.1))
-  (gr_arc (start 269.24 30.48) (mid 271.036051 31.223949) (end 271.78 33.02) (layer "Edge.Cuts") (width 0.1))
-  (gr_arc (start 30.48 144.78) (mid 28.683949 144.036051) (end 27.94 142.24) (layer "Edge.Cuts") (width 0.1))
-  (gr_line (start 27.94 142.24) (end 27.94 33.02) (layer "Edge.Cuts") (width 0.1))
-  (gr_line (start 271.78 33.02) (end 271.78 142.24) (layer "Edge.Cuts") (width 0.1))
-  (gr_text "243.84mm\n" (at 156.21 158.75) (layer "Eco1.User")
+  (gr_arc (start 30.48 142.729949) (mid 28.683949 141.986) (end 27.94 140.189949) (layer "Edge.Cuts") (width 0.1))
+  (gr_arc (start 255.251949 30.48) (mid 257.048 31.223949) (end 257.791949 33.02) (layer "Edge.Cuts") (width 0.1))
+  (gr_line (start 27.94 140.189949) (end 27.94 33.02) (layer "Edge.Cuts") (width 0.1))
+  (gr_line (start 257.791949 33.02) (end 257.791949 140.189949) (layer "Edge.Cuts") (width 0.1))
+  (gr_text "229.852mm\n" (at 152.654 158.496) (layer "Eco1.User")
     (effects (font (size 3 3) (thickness 0.5)))
   )
-  (gr_text "114.30mm" (at 294.64 88.9) (layer "Eco1.User")
+  (gr_text "112.25mm" (at 294.64 88.9) (layer "Eco1.User")
     (effects (font (size 3 3) (thickness 0.5)))
   )
