File: switchplate.kicad_pcb (KiCad board)
At the start: 2 copper layers, 243.8 x 81.3 mm, 4 parts

Commit message: update switchplate
Parts:
- removed the REF** at (251.5, 83.8)
- removed the REF** at (48.3, 83.8)
- removed the REF** at (48.3, 124.5)
- removed the REF** at (251.5, 124.5)
- added REF**: M2_Hole_TH, kbd:M2_Hole_TH, F.Cu at (238.1, 85.0)
- added REF**: M2_Hole_TH, kbd:M2_Hole_TH, F.Cu at (47.6, 123.0)
- added REF**: M2_Hole_TH, kbd:M2_Hole_TH, F.Cu at (47.6, 85.0)
- added REF**: M2_Hole_TH, kbd:M2_Hole_TH, F.Cu at (238.1, 123.1)
Other:
- board size 243.8 x 81.3 mm -> 229.9 x 77.3 mm
- board text added: "229.852mm"
- board text added: "77.274mm"
- board text removed: "243.84mm"
- board text removed: "81.28mm"
